Commit message: got robot arm control working, and added vision processing node for cart

File: cart/cart_description/urdf/cart.xacro (robot description, xacro)
@@ -6,11 +6,11 @@
   <xacro:property name="chassis_length" value="0.3" />
   <xacro:property name="chassis_height" value="0.05" />
-  <xacro:property name="chassis_mass" value="0.5" />
+  <xacro:property name="chassis_mass" value="0.2" />
   <xacro:property name="rear_wheel_radius" value="0.05" />
   <xacro:property name="rear_wheel_thickness" value="0.025" />
   <xacro:property name="rear_wheel_mass" value="0.1" />
   <xacro:property name="rear_wheel_buffer" value="0.01" />
-  <xacro:property name="front_wheel_radius" value="0.01" />
-  <xacro:property name="front_wheel_mass" value="0.01" />
+  <xacro:property name="front_wheel_radius" value="0.02" />
+  <xacro:property name="front_wheel_mass" value="0.0" />
   <xacro:property name="lidar_height" value="0.05" />
   <xacro:property name="lidar_diameter" value="0.07" />
@@ -52,5 +52,5 @@
       <origin xyz="0 0 0" rpy="0 0 0"/>
       <mass value="${rear_wheel_mass}"/>
-      <xacro:cylinder_inertia m="${rear_wheel_mass}" r="${rear_wheel_radius}" h="${rear_wheel_thickness}"/>
+      <xacro:cylinder_inertia m="${rear_wheel_mass}" r="${rear_wheel_radius / 2}" h="${rear_wheel_thickness}"/>
     </inertial>
     <surface>
@@ -79,5 +79,5 @@
       <origin xyz="0 0 0" rpy="0 0 0"/>
       <mass value="${rear_wheel_mass}"/>
-      <xacro:cylinder_inertia m="${rear_wheel_mass}" r="${rear_wheel_radius}" h="${rear_wheel_thickness}"/>
+      <xacro:cylinder_inertia m="${rear_wheel_mass}" r="${rear_wheel_radius / 2}" h="${rear_wheel_thickness}"/>
     </inertial>
     <surface>
@@ -156,5 +156,6 @@
     <parent link="chassis"/>
     <axis xyz="0 0 -1"/>
-    <dynamics damping="0.0" friction="0.2"/>
+    <limit effort="0.5" velocity="20" />
+    <dynamics damping="0.0" friction="0.05"/>
   </joint>
   <joint type="continuous" name="left_wheel_hinge">
@@ -163,5 +164,6 @@
     <parent link="chassis"/>
     <axis xyz="0 0 1"/>
-    <dynamics damping="0.0" friction="0.2"/>
+    <limit effort="0.5" velocity="20" />
+    <dynamics damping="0.0" friction="0.05"/>
   </joint>
   <joint type="fixed" name="front_wheel_hinge">
